File: KiCad_ETDBR/KiCad_ETDBR.kicad_pcb (KiCad board)
At the start: 2 copper layers, 35 x 50 mm, 15 parts, among them J1 Conn_01x01_Pin, J2 Conn_02x08_Top_Bottom

Commit message: edits on single digit pcb in kicad with gerber
Routing:
- net Net-(J2-Pin_16): track 48.7 -> 44.0 mm
- net Net-(J2-Pin_9): track 37.7 -> 38.3 mm
