File: KiCad_ETDBR/KiCad_ETDBR.kicad_sch (KiCad schematic)
At the start: 11 parts, among them J1 Conn_01x01_Pin, J2 Conn_02x08_Top_Bottom

Commit message: edits on single digit pcb in kicad with gerber
Changed lines of the file:
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@@
 		(on_board yes)
 		(dnp no)
+		(fields_autoplaced yes)
 		(property "Reference" "U2"
-			(at 101.854 76.2 0)
+			(at 101.6 71.12 0)
 			(effects
 				(font
@@
 			)
 		)
+		(pin "-1"
+		)
+		(pin "8"
+		)
+		(pin "7"
+		)
+		(pin "1"
+		)
+		(pin "-8"
+		)
+		(pin "-6"
+		)
+		(pin "2"
+		)
+		(pin "-5"
+		)
+		(pin "5"
+		)
+		(pin "-3"
+		)
+		(pin "4"
+		)
 		(pin "-7"
 		)
@@
 		(pin "-4"
 		)
-		(pin "5"
-		)
-		(pin "-5"
+		(pin "6"
 		)
 		(pin "3"
 		)
-		(pin "1"
-		)
-		(pin "2"
-		)
-		(pin "-8"
-		)
-		(pin "-1"
-		)
-		(pin "-6"
-		)
-		(pin "-3"
-		)
-		(pin "6"
-		)
-		(pin "7"
-		)
-		(pin "8"
-		)
-		(pin "4"
-		)
 		(instances
